File: Franzininho-RP2040.sch (KiCad schematic (older format))
At the start: 32 parts

Commit message: Adição de conector SWD, definição de pinos e pequenas correções
Parts:
- removed J?: Conn_01x16, symbol Connector_Generic:Conn_01x16
- added D?: D_Schottky, symbol Device:D_Schottky
- added J?: Conn_01x03, symbol Connector_Generic:Conn_01x03
- added J? (x2): Conn_01x17, symbol Connector_Generic:Conn_01x17
- added R? (x2): 27, symbol Device:R
- C?: value 10u -> 100n
- C? (x2): value C -> 27p
- R?: value R -> 1k
- R?: value R -> 10k
- Y?: value Crystal -> 12MHz
Connections:
- net labels added: +5V, GPIO0, GPIO1, GPIO10, GPIO11, GPIO12, GPIO13, GPIO14, GPIO15, GPIO16, GPIO17, GPIO18, GPIO19, GPIO2, GPIO20, GPIO21, GPIO22, GPIO23, GPIO24, GPIO25, GPIO26_ADC0, GPIO27_ADC1, GPIO28_ADC2, GPIO29_ADC3, GPIO3, GPIO4, GPIO5, GPIO6, GPIO7, GPIO8, GPIO9, SWCLK, SWDCLK, SWDIO, ~RESET, ~USB_BOOT
- net labels removed: D10, D11, D12, D13, D4, D5, D6, D9, \RESET
- wire segments 176 -> 227
Other:
- note added: "Crystal oscillator"
- note added: "Reset button"
- note added: "SWD"
- note removed: "Crystal Oscillator"
- note removed: "Reset\nbutton"
- moved on the sheet: C?, D?, J?, R?, SW?, U?

Commit message: Anotação de esquemático
Parts:
- gave numbers to parts that had none: 37
Other:
- moved on the sheet: C12, C13, R4, R8, SW1, Y1

Commit message: ERC e correções
Connections:
- net SWCLK is gone; now on net SWDCLK: U1.24 (SWCLK)
Changed lines of the file:
@@
 	775  5025 1275 5025
-Wire Wire Line
-	775  6325 1275 6325
 Wire Wire Line
 	775  6425 1275 6425
@@
 Wire Wire Line
 	5700 3950 6300 3950
-Text Notes 5775 6925 0    197  ~ 0
-SWD
 $Comp
 L Connector_Generic:Conn_01x03 J3
@@
 	-1   0    0    -1
 $EndComp
-Text Label 775  6325 0    50   ~ 0
-SWCLK
 Text Label 775  6425 0    50   ~ 0
 SWDIO
 Wire Wire Line
-	6375 7250 6050 7250
-Wire Wire Line
 	6375 7450 6050 7450
-Text Label 6375 7250 2    50   ~ 0
-SWDCLK
 Text Label 6375 7450 2    50   ~ 0
 SWDIO
@@
 Wire Notes Line
 	8976 484  8976 6543
+Wire Wire Line
+	6375 7250 6050 7250
+Text Label 6373 7250 2    50   ~ 0
+SWDCLK
+Text Notes 5775 6925 0    197  ~ 0
+SWD
+Wire Wire Line
+	775  6325 1275 6325
+Text Label 775  6325 0    50   ~ 0
+SWDCLK
 $EndSCHEMATC

Commit message: Adição de nomes de nets + pequenas melhorias e correções
Parts:
- removed J3: Conn_01x03, symbol Connector_Generic:Conn_01x03
- removed SW1: SW_MEC_5G, symbol Switch:SW_MEC_5G
- added J3: Conn_01x04, Connector_PinHeader_2.54mm:PinHeader_1x04_P2.54mm_Vertical, symbol Connector_Generic:Conn_01x04
- added SW1: SW_Push, Button_Switch_SMD:SW_SPST_B3U-1000P, symbol Switch:SW_Push
- C1, C10, C11, C16, C2, C3, C4, C5, C6, C7, C8, C9: footprint (none) -> Capacitor_SMD:C_0402_1005Metric_Pad0.74x0.62mm_HandSolder
- C12, C13: footprint (none) -> Capacitor_SMD:C_0603_1608Metric_Pad1.08x0.95mm_HandSolder
- C14, C15: footprint (none) -> Capacitor_SMD:C_1206_3216Metric_Pad1.33x1.80mm_HandSolder
- D1: footprint (none) -> Diode_SMD:D_SOD-123
- D2, D3: footprint (none) -> LED_SMD:LED_0805_2012Metric_Pad1.15x1.40mm_HandSolder
- J1: footprint (none) -> Connector_USB:USB_Micro-B_Amphenol_10118194_Horizontal
- J2: footprint (none) -> Connector_PinHeader_2.54mm:PinHeader_1x02_P2.54mm_Vertical
- J4, J5: footprint (none) -> Connector_PinHeader_2.54mm:PinHeader_1x17_P2.54mm_Vertical
- R1, R2, R3, R4, R5: footprint (none) -> Resistor_SMD:R_0402_1005Metric_Pad0.72x0.64mm_HandSolder
- R6, R7, R8: footprint (none) -> Resistor_SMD:R_0805_2012Metric_Pad1.20x1.40mm_HandSolder
- U1: footprint QFN40P695X695X90-57T320N -> Biblioteca de footprints:QFN40P695X695X90-57T320N
- Y1: footprint (none) -> Crystal:Crystal_SMD_2520-4Pin_2.5x2.0mm
Connections:
- net +1V1: no longer C1.2, C10.2, C11.2, C12.2, C13.2, C14.2, C15.2, C16.2, C2.2, C3.2, C4.2, C5.2, C6.2, C7.2, C8.2, C9.2, D2.1 (K), D3.1 (K), J1.5 (GND), J1.6 (Shield), J2.2 (Pin_2), J4.2 (Pin_2), J5.2 (Pin_2), J5.3 (Pin_3), U1.19 (TESTEN), U1.57 (PAD), U2.1 (GND), U3.4 (GND)
- net +3V3: now also J3.1 (Pin_1)
- net SWDIO: now also J3.3 (Pin_3)
- net ~RESET: now also SW1.2
- net XOUT_R: now reaches C13.1, R4.2, Y1.2
- net POWER_LED: now reaches D2.2 (A), R6.1
- net USER_LED: now reaches D3.2 (A), R7.1
- net SWDCLK renamed SWCLK
- net SWCLK: now also J3.2 (Pin_2)
- new net GND: C1.2, C10.2, C11.2, C12.2, C13.2, C14.2, C15.2, C16.2, C2.2, C3.2, C4.2, C5.2, C6.2, C7.2, C8.2, C9.2, D2.1 (K), D3.1 (K), J1.5 (GND), J1.6 (Shield), J2.2 (Pin_2), J3.4 (Pin_4), J4.2 (Pin_2), J5.2 (Pin_2), J5.3 (Pin_3), SW1.1, U1.19 (TESTEN), U1.57 (PAD), U2.1 (GND), U3.4 (GND)
Other:
- moved on the sheet: C12, C13, D3, R4, R6, R7, Y1

Commit message: Adição de modelos 3D e melhorias
Parts:
- removed J2: Conn_01x02, Connector_PinHeader_2.54mm:PinHeader_1x02_P2.54mm_Vertical, symbol Connector_Generic:Conn_01x02
- removed U2: NCP1117-3.3_SOT223, Package_TO_SOT_SMD:SOT-223-3_TabPin2, symbol Regulator_Linear:NCP1117-3.3_SOT223
- added H1, H2, H3, H4: MountingHole, MountingHole:MountingHole_2.2mm_M2, symbol Mechanical:MountingHole
- added SW2: SW_Push, Button_Switch_SMD:SW_SPST_PTS810, symbol Switch:SW_Push
- added U2: XC6206P332MR, Package_TO_SOT_SMD:SOT-23, symbol Regulator_Linear:XC6206PxxxMR
- C12, C13: footprint Capacitor_SMD:C_0603_1608Metric_Pad1.08x0.95mm_HandSolder -> Capacitor_SMD:C_0402_1005Metric_Pad0.74x0.62mm_HandSolder
- SW1: footprint Button_Switch_SMD:SW_SPST_B3U-1000P -> Button_Switch_SMD:SW_SPST_PTS810
Connections:
- net +3V3: now also U2.2 (VO)
- net +5V: now also U2.3 (VI)
- net GND: now also SW2.1, U2.1 (GND)
- net ~RESET: now also SW2.2; no longer SW1.2
- net ~USB_BOOT: now also SW1.2
Other:
- moved on the sheet: C1, C10, C11, C16, C2, C3, C4, C5, C6, C7, C8, C9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
